File: Hardware/PCB/vcapf/vcapf.kicad_sch (KiCad schematic)
At the start: 60 parts, among them J1 Synth_power_2x5

Commit message: Post breadboard tweaks; layout
Parts:
- removed C2, C4, C? (x6): 100nF, ao_tht:C_Disc_D3.0mm_W1.6mm_P2.50mm, symbol ao_symbols:C
- removed C?: 4.7nF, ao_tht:C_Disc_D3.0mm_W1.6mm_P2.50mm, symbol ao_symbols:C
- removed D?: 1N4148, ao_tht:D_DO-35_SOD27_P7.62mm_Horizontal, symbol ao_symbols:1N4148
- removed Q? (x2): 2N3906, ao_tht:TO-92_Inline_Wide, symbol ao_symbols:2N3906
- removed R?: 15k, ao_tht:R_Axial_DIN0207_L6.3mm_D2.5mm_P10.16mm_Horizontal, symbol ao_symbols:R
- removed R? (x7): 100k, ao_tht:R_Axial_DIN0207_L6.3mm_D2.5mm_P10.16mm_Horizontal, symbol ao_symbols:R
- removed R?: 4.7k, ao_tht:R_Axial_DIN0207_L6.3mm_D2.5mm_P10.16mm_Horizontal, symbol ao_symbols:R
- removed R?: 470k, ao_tht:R_Axial_DIN0207_L6.3mm_D2.5mm_P10.16mm_Horizontal, symbol ao_symbols:R
- removed R? (x2): 6.8k, ao_tht:R_Axial_DIN0207_L6.3mm_D2.5mm_P10.16mm_Horizontal, symbol ao_symbols:R
- removed R? (x2): 1k, ao_tht:R_Axial_DIN0207_L6.3mm_D2.5mm_P10.16mm_Horizontal, symbol ao_symbols:R
- removed R? (x4): 620R, ao_tht:R_Axial_DIN0207_L6.3mm_D2.5mm_P10.16mm_Horizontal, symbol ao_symbols:R
- removed R?: 1.8k, ao_tht:R_Axial_DIN0207_L6.3mm_D2.5mm_P10.16mm_Horizontal, symbol ao_symbols:R
- removed R? (x4): 30k, ao_tht:R_Axial_DIN0207_L6.3mm_D2.5mm_P10.16mm_Horizontal, symbol ao_symbols:R
- removed R? (x2): 7.5k, ao_tht:R_Axial_DIN0207_L6.3mm_D2.5mm_P10.16mm_Horizontal, symbol ao_symbols:R
- removed R?: (no value), ao_tht:R_Axial_DIN0207_L6.3mm_D2.5mm_P10.16mm_Horizontal, symbol ao_symbols:R
- removed R?: 10k, ao_tht:R_Axial_DIN0207_L6.3mm_D2.5mm_P10.16mm_Horizontal, symbol ao_symbols:R
- removed U? (x5): TL074, ao_tht:DIP-14_W7.62mm_Socket_LongPads, symbol ao_symbols:TL074
- removed U? (x5): LM13700, ao_tht:DIP-16_W7.62mm_Socket_LongPads, symbol ao_symbols:LM13700
- removed U? (x3): TL072, ao_tht:DIP-8_W7.62mm_Socket_LongPads, symbol ao_symbols:TL072
- added GRAF1: Holes, vcapf:vcapf_panel_holes, symbol ao_symbols:Graphic
- added GRAF2: CC0 logo, ao_tht:CC0_logo, symbol ao_symbols:Graphic
- added GRAF3: AO logo, ao_tht:analogoutput, symbol ao_symbols:Graphic
- added H1, H2, H3, H4: MountingHole, ao_tht:MountingHole_3.2mm_M3, symbol ao_symbols:MountingHole
- added J2, J3, J6, J7: AudioJack2, ao_tht:Jack_6.35mm_PJ_629HAN_slots, symbol ao_symbols:AudioJack2
- added J4: Conn_01x05, Connector_PinSocket_2.54mm:PinSocket_1x05_P2.54mm_Vertical, symbol Connector_Generic:Conn_01x05
- added J5: Conn_01x05, Connector_PinHeader_2.54mm:PinHeader_1x05_P2.54mm_Vertical, symbol Connector_Generic:Conn_01x05
- added R25, R26: 100k, ao_tht:R_Axial_DIN0207_L6.3mm_D2.5mm_P10.16mm_Horizontal, symbol ao_symbols:R
- added R27, R28: 1k, ao_tht:R_Axial_DIN0207_L6.3mm_D2.5mm_P10.16mm_Horizontal, symbol ao_symbols:R
- TP1, TP3: value TestPoint -> (none)
- TP2: value TestPoint -> (none); footprint ao_tht:TestPoint_THTPad_D1.5mm_Drill0.7mm -> ao_tht:TestPoint_THTPad_1.5x1.5mm_Drill0.7mm
- renumbered C3 to C2
Connections:
- net GND: now also J4.5 (Pin_5)
- new net: J6.S, R27.2
- new net: J7.S, R28.2
- new net 1POLE_OUT_J: J5.3 (Pin_3), R25.1, R27.1
- new net 2POLE_OUT_J: J5.4 (Pin_4), R26.1, R28.1
- new net CV_J: J3.S, J5.2 (Pin_2)
- new net GND1: J2.T, J3.T, J5.5 (Pin_5), J6.T, J7.T, R25.2, R26.2
- new net INPUT_J: J2.S, J5.1 (Pin_1)
- new net Main PCB/1POLE_OUT: J4.3 (Pin_3)
- new net Main PCB/2POLE_OUT: J4.4 (Pin_4)
- new net Main PCB/CV_IN: J4.2 (Pin_2)
- new net Main PCB/INPUT: J4.1 (Pin_1)
- no-connect marks 6 -> 0
Other:
- added sheet Main PCB (vcapf_main.kicad_sch)
- note removed: "2 pole LPF"
- note removed: "At 0 freq: Input - 2 * LP1 + inversion = 0° phase shift"
- note removed: "At 0 freq: Input - 4 * LP1 + 4 * LP2 + 2 * inversion = 0° phase shift"
- note removed: "Exponential converter"
- note removed: "Per LM13700 datasheet, f_0 = R_A g_m / ((R+R_A)2πC) R_A = 620 R = 100k g_m ~ 9600 µS at I_ABC = 500 µA (~ 19.2I_ABC). f0 ~ 10/C Hz with C in µF."
- note removed: "Pole mixing"

Commit message: Net labels, panel
Parts:
- TP1: value (none) -> +12V
- TP2: value (none) -> GND
- TP3: value (none) -> -12V
Connections:
- net 1P OUT: now reaches J6.S, R27.2
- net 2P OUT: now reaches J7.S, R28.2
Changed lines of the file:
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@@
     (effects (font (size 2.54 2.54)) (justify left bottom))
+  )
+  (label "2P OUT" (at 214.63 88.9 270)
+    (effects (font (size 1.27 1.27)) (justify right bottom))
+  )
+  (label "1P OUT" (at 214.63 69.85 270)
+    (effects (font (size 1.27 1.27)) (justify right bottom))
   )
   (label "CV_J" (at 186.69 78.74 0)
@@
       (effects (font (size 1.27 1.27)) (justify right))
     )
-    (property "Value" "" (id 1) (at 43.053 198.0442 0)
+    (property "Value" "+12V" (id 1) (at 43.053 198.0442 0)
       (effects (font (size 1.27 1.27)) (justify right))
     )
@@
       (effects (font (size 1.27 1.27)) (justify left))
     )
-    (property "Value" "" (id 1) (at 71.247 192.7102 0)
+    (property "Value" "-12V" (id 1) (at 71.247 192.7102 0)
       (effects (font (size 1.27 1.27)) (justify left))
     )
@@
       (effects (font (size 1.27 1.27)) (justify left))
     )
-    (property "Value" "" (id 1) (at 57.277 192.7102 0)
-      (effects (font (size 1.27 1.27)) (justify left))
-    )
+    (property "Value" "GND" (id 1) (at 57.277 192.7102 0)
+      (effects (font (size 1.27 1.27)) (justify left))
+    )

Commit message: Pre fab tweaks, unreverse jacks, Gerbers
Parts:
- added B1: Board, ao_tht:Board_Marker, symbol ao_symbols:Board
- renumbered R25 to R1, R26 to R2, R27 to R3, R28 to R4
Connections:
- net 1P OUT: now also J6.T; no longer J6.S
- net 2P OUT: now also J7.T; no longer J7.S
- net 2POLE_OUT_J: now also J5.2 (Pin_2); no longer J5.4 (Pin_4)
- net CV_J: now also J3.T, J5.4 (Pin_4); no longer J3.S, J5.2 (Pin_2)
- net GND: now also J4.1 (Pin_1); no longer J4.5 (Pin_5)
- net GND1: now also J2.S, J3.S, J5.1 (Pin_1), J6.S, J7.S; no longer J2.T, J3.T, J5.5 (Pin_5), J6.T, J7.T
- net INPUT_J: now also J2.T, J5.5 (Pin_5); no longer J2.S, J5.1 (Pin_1)
- net Main PCB/2POLE_OUT: now also J4.2 (Pin_2); no longer J4.4 (Pin_4)
- net Main PCB/CV_IN: now also J4.4 (Pin_4); no longer J4.2 (Pin_2)
- net Main PCB/INPUT: now also J4.5 (Pin_5); no longer J4.1 (Pin_1)
Other:
- moved on the sheet: J2, J3, J5, J6, J7

Commit message: Post fab updates
Parts:
- J4: SKU (none) -> A-196 (cut); Vendor (none) -> Tayda
- J5: SKU (none) -> A-197 (cut); Vendor (none) -> Tayda
Changed lines of the file:
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@@
+      (effects (font (size 1.27 1.27)) hide)
+    )
+    (property "Description" "Electrolytic capacitor, 2.5 mm pitch" (id 6) (at 118.11 172.72 0)
       (effects (font (size 1.27 1.27)) hide)
     )
@@
       (effects (font (size 1.27 1.27)) hide)
     )
+    (property "Description" "Electrolytic capacitor, 2.5 mm pitch" (id 6) (at 118.11 180.34 0)
+      (effects (font (size 1.27 1.27)) hide)
+    )
     (pin "1")
     (pin "2")
@@
     )
     (property "Vendor" "Tayda" (id 4) (at 203.2 93.98 0)
+      (effects (font (size 1.27 1.27)) hide)
+    )
+    (property "Description" "1/4 watt resistor, metal film" (id 5) (at 203.2 93.98 0)
       (effects (font (size 1.27 1.27)) hide)
     )
@@
       (effects (font (size 1.27 1.27)) hide)
     )
+    (property "Description" "1/4 watt resistor, metal film" (id 5) (at 208.28 69.85 0)
+      (effects (font (size 1.27 1.27)) hide)
+    )
     (pin "1")
     (pin "2")
@@
       (effects (font (size 1.27 1.27)) hide)
     )
+    (property "Description" "5 pin socket, 2.5 mm pitch" (id 4) (at 161.29 81.28 0)
+      (effects (font (size 1.27 1.27)) hide)
+    )
+    (property "SKU" "A-196 (cut)" (id 5) (at 161.29 81.28 0)
+      (effects (font (size 1.27 1.27)) hide)
+    )
+    (property "Vendor" "Tayda" (id 6) (at 161.29 81.28 0)
+      (effects (font (size 1.27 1.27)) hide)
+    )
     (pin "1")
     (pin "2")
@@
       (effects (font (size 1.27 1.27)) hide)
     )
+    (property "Description" "1/4\" audio jack, vertical" (id 6) (at 96.52 88.9 0)
+      (effects (font (size 1.27 1.27)) hide)
+    )
     (pin "S")
     (pin "T")
@@
       (effects (font (size 1.27 1.27)) hide)
     )
+    (property "Description" "1/4\" audio jack, vertical" (id 6) (at 223.52 88.9 0)
+      (effects (font (size 1.27 1.27)) hide)
+    )
     (pin "S")
     (pin "T")
@@
     )
     (property "Vendor" "Tayda" (id 4) (at 203.2 74.93 0)
+      (effects (font (size 1.27 1.27)) hide)
+    )
+    (property "Description" "1/4 watt resistor, metal film" (id 5) (at 203.2 74.93 0)
       (effects (font (size 1.27 1.27)) hide)
     )
@@
       (effects (font (size 1.27 1.27)) hide)
     )
+    (property "Description" "1/4 watt resistor, metal film" (id 5) (at 208.28 88.9 0)
+      (effects (font (size 1.27 1.27)) hide)
+    )
     (pin "1")
     (pin "2")
@@
     )
     (property "SKU" "A-1121" (id 5) (at 223.52 69.85 0)
+      (effects (font (size 1.27 1.27)) hide)
+    )
+    (property "Description" "1/4\" audio jack, vertical" (id 6) (at 223.52 69.85 0)
       (effects (font (size 1.27 1.27)) hide)
     )
@@
       (effects (font (size 1.27 1.27)) hide)
     )
+    (property "Description" "5 pin header, 2.5 mm pitch" (id 4) (at 179.07 81.28 0)
+      (effects (font (size 1.27 1.27)) hide)
+    )
+    (property "SKU" "A-197 (cut)" (id 5) (at 179.07 81.28 0)
+      (effects (font (size 1.27 1.27)) hide)
+    )
+    (property "Vendor" "Tayda" (id 6) (at 179.07 81.28 0)
+      (effects (font (size 1.27 1.27)) hide)
+    )
     (pin "1")
     (pin "2")
@@
       (effects (font (size 1.27 1.27)) hide)
     )
+    (property "Description" "1/4\" audio jack, vertical" (id 6) (at 96.52 74.93 0)
+      (effects (font (size 1.27 1.27)) hide)
+    )
